File: schematics/sensor/sensor-sm.sch (EAGLE design)
At the start: 22 parts, among them IC1 STM8S208S4, IC2 LP2950CDT-5.0, Q1 8MHz, U1 MCP2551SN

Commit message: Add latest changes to the home-automation project
Parts:
- removed CAN: CWF-4R, connector:CWF-4R
- added D1: GS1J, diode:GF1
- added NUP2105L: NUP2105L, transistor:NUP2105L
- added X1, X2: YH-55-10, con-wenzhou-yihua:YH-55-10
- LED1, LED2, PWR: device led:LEDSML0805 -> led:LEDSML1206
Connections:
- removed net N$2: CAN.P$4, U1>NAME.CANL
- new net N$10: C5.1, C8.+, D1.C, IC2.IN
- new net N$9: NUP2105L.P$2, U1>NAME.CANH, X1.3, X2.3
- net GND: now also NUP2105L.P$3, X1.5, X2.5; no longer CAN.P$2
- net N$4: now also NUP2105L.P$1, U1>NAME.CANL, X1.4, X2.4; no longer CAN.P$3, U1>NAME.CANH
- net V_CAN: now also D1.A, X1.2, X2.2; no longer C5.1, C8.+, CAN.P$1, IC2.IN
